Commit message: Small fix on collision pose

File: softkinetic_camera/urdf/senz3d.urdf.xacro (robot description, xacro)
@@ -20,8 +20,8 @@
       </visual>
       <collision>
-        <origin xyz="-0.01 0.0 0.0" rpy="0 0 0"/>
+        <origin xyz="-0.015 0.0 0.0" rpy="0 0 0"/>
         <geometry>
-        <box size="0.04 0.11 0.04"/>
-      </geometry>
+          <box size="0.04 0.11 0.04"/>
+        </geometry>
       </collision>
       <inertial>

Commit message: Change tf frames to mimick Kinect and Asus cameras: make the RGB frame link the root of the camera tree

File: softkinetic_camera/urdf/senz3d.urdf.xacro (robot description, xacro)
@@ -6,7 +6,23 @@
   <xacro:property name="M_PI" value="3.14159265359"/>
   <xacro:macro name="sensor_senz3d" params="parent name *origin">
-    <joint name="${name}_joint" type="fixed">
+    <!-- Add RGB and RGB optical frames -->
+    <joint name="${name}_rgb_joint" type="fixed">
+      <!-- RGB joint is the base of the tf tree, as for Kinect -->
       <insert_block name="origin"/>
       <parent link="${parent}"/>
+      <child link="${name}_rgb_frame"/>
+    </joint>
+    <link name="${name}_rgb_frame"/>
+    <joint name="${name}_rgb_optical_joint" type="fixed">
+      <origin xyz="0.0 0.0 0.0" rpy="${-M_PI/2} 0.0 ${-M_PI/2}"/>
+      <parent link="${name}_rgb_frame"/>
+      <child link="${name}_rgb_optical_frame"/>
+    </joint>
+    <link name="${name}_rgb_optical_frame"/>
+    <!-- Senz3D camera link with the visual, inertia and collision models -->
+    <!-- Mimicking Kinect and Asus cameras, it's a child of RGB frame link -->
+    <joint name="${name}_joint" type="fixed">
+      <origin xyz="0.0 -0.013 0.0" rpy="0.0 0.0 0.0"/>
+      <parent link="${name}_rgb_frame"/>
       <child link="${name}_link"/>
     </joint>
@@ -33,20 +49,8 @@
       </inertial>
     </link>
-    <!-- Add frames for RGB and depth optical axes -->
-    <joint name="${name}_rgb_joint" type="fixed">
-      <origin xyz="0.0 0.0125 0.0" rpy="0.0 0.0 0.0"/>
-      <parent link="${name}_link"/>
-      <child link="${name}_rgb_frame"/>
-    </joint>
-    <link name="${name}_rgb_frame"/>
-    <joint name="${name}_rgb_optical_joint" type="fixed">
-      <origin xyz="0.0 0.0 0.0" rpy="${-M_PI/2} 0.0 ${-M_PI/2}"/>
+    <!-- Depth and depth optical frames, also childs of RGB frame link -->
+    <joint name="${name}_depth_joint" type="fixed">
+      <origin xyz="0.0 -0.026 0.0" rpy="0.0 0.0 0.0"/>
       <parent link="${name}_rgb_frame"/>
-      <child link="${name}_rgb_optical_frame"/>
-    </joint>
-    <link name="${name}_rgb_optical_frame"/>
-    <joint name="${name}_depth_joint" type="fixed">
-      <origin xyz="0.0 -0.0125 0.0" rpy="0.0 0.0 0.0"/>
-      <parent link="${name}_link"/>
       <child link="${name}_depth_frame"/>
     </joint>

Commit message: Minor changes on camera visual and collision dimensions

File: softkinetic_camera/urdf/senz3d.urdf.xacro (robot description, xacro)
@@ -29,8 +29,8 @@
     <link name="${name}_link">
       <visual>
-        <origin xyz="-0.01 0.0 0.0" rpy="${-M_PI/2} -${M_PI} ${-M_PI/2}"/>
+        <origin xyz="-0.015 0.0 0.0" rpy="${-M_PI/2} -${M_PI} ${-M_PI/2}"/>
         <geometry>
           <!-- As we don't have a Senz3D mesh, use a deformed Asus Xtion Pro instead -->
-          <mesh filename="package://softkinetic_camera/meshes/asus_xtion_pro_live.dae" scale="0.0006 0.0015 0.001"/>
+          <mesh filename="package://softkinetic_camera/meshes/asus_xtion_pro_live.dae" scale="0.0006 0.0015 0.0006"/>
         </geometry>
       </visual>
@@ -38,5 +38,5 @@
         <origin xyz="-0.015 0.0 0.0" rpy="0 0 0"/>
         <geometry>
-          <box size="0.04 0.11 0.04"/>
+          <box size="0.03 0.11 0.04"/>
         </geometry>
       </collision>
